Commit message: working examples added

File: URDF import examples/robots_library/cheetah/urdf/cheetah.urdf (robot description, URDF)
Before this commit: robot cheetah, 25 links, 24 joints
Joints:
- removed joint trunk_to_trunk_inertia
- added joint trunk_to_trunk_inertia_floating: type revoluteeee, parent trunk, child trunk_interia, origin xyz=0 0 0 rpy=0 0 0, limit lower=-0.872664625997 upper=1.0471975512 effort=20 velocity=10.6
